Commit message: Updated urdf with GPS + IMU

File: scout_description/urdf/scout_v2.urdf (robot description, URDF)
Before this commit: robot scout_v2, 7 links, 6 joints
Links:
- added link gps_link; visual box size=0.1 0.1 0.1
- added link imu_link, mass 0.1; collision box size=0.1 0.1 0.1; visual box size=0.1 0.1 0.1
- link base_link: geometry collision box size=0.15416666666666667 0.627 0.06999999999999999; collision box size=0.925 0.38 0.21
- link front_left_wheel_link: geometry collision cylinder length=0.11653 radius=0.16459; visual mesh filename=file:///home/emanuel/ros2_ws/install/scout_description/shar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
- link front_right_wheel_link: geometry collision cylinder length=0.11653 radius=0.16459; visual mesh filename=file:///home/emanuel/ros2_ws/install/scout_description/shar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
- link rear_left_wheel_link: geometry collision cylinder length=0.11653 radius=0.16459; visual mesh filename=file:///home/emanuel/ros2_ws/install/scout_description/shar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
- link rear_right_wheel_link: geometry collision cylinder length=0.11653 radius=0.16459; visual mesh filename=file:///home/emanuel/ros2_ws/install/scout_description/shar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
Joints:
- added joint gps_joint: type fixed, parent base_link, child gps_link, origin xyz=0 0 0 rpy=0 0 0
- added joint imu_joint: type fixed, parent base_link, child imu_link, origin xyz=0 0 0.01
- joint base_footprint_joint: type continuous -> fixed
- joint front_right_wheel: origin xyz=0.249 -0.29153 -0.0702 rpy=3.14 0 0 -> xyz=0.249 -0.29153 -0.0702 rpy=3.141592653589793 0 0
- joint rear_right_wheel: origin xyz=-0.249 -0.29153 -0.0702 rpy=3.14 0 0 -> xyz=-0.249 -0.29153 -0.0702 rpy=3.141592653589793 0 0

File: scout_description/urdf/scout_v2.xacro (robot description, xacro)
@@ -16,4 +16,11 @@
     <xacro:property name="wheel_length" value="1.1653e-01" />
     <xacro:property name="wheel_radius" value="1.6459e-01" />
+    <xacro:macro name="box_inertia" params="m w h d">
+    <inertial>
+      <origin xyz="0 0 0" rpy="${pi/2} 0 ${pi/2}"/>
+      <mass value="${m}"/>
+      <inertia ixx="${(m/12) * (h*h + d*d)}" ixy="0.0" ixz="0.0" iyy="${(m/12) * (w*w + d*d)}" iyz="0.0" izz="${(m/12) * (w*w + h*h)}"/>
+    </inertial>
+    </xacro:macro>
     <!-- Base link -->
     <link name="base_link">
@@ -70,3 +77,116 @@
         <origin xyz="${-wheelbase/2} ${-track/2} ${wheel_vertical_offset}" rpy="${pi} 0 0" />
     </xacro:scout_wheel_type2>
+    <link name="gps_link">
+        <visual>
+        <origin xyz="0 0.5 0"/>
+        <geometry>
+            <box size="0.1 0.1 0.1" />
+        </geometry>
+        </visual>
+    </link>
+    <joint name="gps_joint" type="fixed">
+        <origin xyz="0 0 0" rpy="0 0 0" />
+        <parent link="base_link" />
+        <child link="gps_link" />
+    </joint>
+    <gazebo reference="gps_link">
+        <sensor name="gps_sensor" type="gps">
+            <always_on>true</always_on>
+            <update_rate>1.0</update_rate>
+            <plugin name="gps_controller" filename="libgazebo_ros_gps_sensor.so">
+                <ros>
+                    <!-- <namespace>/br</namespace> -->
+                    <remapping>~/out:=/gps/fix</remapping>
+                </ros>
+                <frame_name>gps_link</frame_name>
+            </plugin>
+        </sensor>
+        <material>Gazebo/Grey</material>
+    </gazebo>
+    <link name="imu_link">
+  <visual>
+    <geometry>
+      <box size="0.1 0.1 0.1"/>
+    </geometry>
+  </visual>
+  <collision>
+    <geometry>
+      <box size="0.1 0.1 0.1"/>
+    </geometry>
+  </collision>
+  <xacro:box_inertia m="0.1" w="0.1" d="0.1" h="0.1"/>
+</link>
+<joint name="imu_joint" type="fixed">
+  <parent link="base_link"/>
+  <child link="imu_link"/>
+  <origin xyz="0 0 0.01"/>
+</joint>
+ <gazebo reference="imu_link">
+  <sensor name="imu_sensor" type="imu">
+   <plugin filename="libgazebo_ros_imu_sensor.so" name="imu_plugin">
+      <ros>
+        <namespace>/demo</namespace>
+        <remapping>~/out:=imu</remapping>
+      </ros>
+      <initial_orientation_as_reference>false</initial_orientation_as_reference>
+    </plugin>
+    <always_on>true</always_on>
+    <update_rate>100</update_rate>
+    <visualize>true</visualize>
+    <imu>
+      <angular_velocity>
+        <x>
+          <noise type="gaussian">
+            <mean>0.0</mean>
+            <stddev>2e-4</stddev>
+            <bias_mean>0.0000075</bias_mean>
+            <bias_stddev>0.0000008</bias_stddev>
+          </noise>
+        </x>
+        <y>
+          <noise type="gaussian">
+            <mean>0.0</mean>
+            <stddev>2e-4</stddev>
+            <bias_mean>0.0000075</bias_mean>
+            <bias_stddev>0.0000008</bias_stddev>
+          </noise>
+        </y>
+        <z>
+          <noise type="gaussian">
+            <mean>0.0</mean>
+            <stddev>2e-4</stddev>
+            <bias_mean>0.0000075</bias_mean>
+            <bias_stddev>0.0000008</bias_stddev>
+          </noise>
+        </z>
+      </angular_velocity>
+      <linear_acceleration>
+        <x>
+          <noise type="gaussian">
+            <mean>0.0</mean>
+            <stddev>1.7e-2</stddev>
+            <bias_mean>0.1</bias_mean>
+            <bias_stddev>0.001</bias_stddev>
+          </noise>
+        </x>
+        <y>
+          <noise type="gaussian">
+            <mean>0.0</mean>
+            <stddev>1.7e-2</stddev>
+            <bias_mean>0.1</bias_mean>
+            <bias_stddev>0.001</bias_stddev>
+          </noise>
+        </y>
+        <z>
+          <noise type="gaussian">
+            <mean>0.0</mean>
+            <stddev>1.7e-2</stddev>
+            <bias_mean>0.1</bias_mean>
+            <bias_stddev>0.001</bias_stddev>
+          </noise>
+        </z>
+      </linear_acceleration>
+    </imu>
+  </sensor>
+</gazebo>
 </robot>
